File: PortableRAM-8MB.kicad_sch (KiCad schematic)
At the start: 37 parts, among them J1 RAM Connector, J2 JTAG_Header_2.54mm_1x06, U1 ATF1502ASL, U11 74HC245, U12 74HC245, U2 AS6C8008-55ZIN, U3 AS6C8008-55ZIN, U4 AS6C8008-55ZIN, U5 AS6C8008-55ZIN, U6 AS6C8008-55ZIN, U7 AS6C8008-55ZIN, U8 AS6C8008-55ZIN, U9 AS6C8008-55ZIN

Commit message: v3 board: MODEL jumper, bank LEDs, pull-down resistors, sequential population
- MODEL jumper (JP1): open=M5120 full 8MB, closed=M5126 cap at 6MB to
  avoid SLOT_CS0 conflict with backlit display controller
- 4 green latching LEDs (D1–D4) — CPLD registered macrocell latches ON
  when each 2MB bank is confirmed at boot; power-cycle clears
- 16× 10KΩ pull-downs (R5–R20) on SD0–SD15 to prevent ghost RAM reads
  on unpopulated banks
- Sequential bank population: U1+U5=2MB, U2+U6=4MB, U3+U7=6MB, U4+U8=8MB
  (no SIZE jumper needed)
- Firmware recompiled for v3 (WinCUPL + Wine, prjbureau SVF) 2026-07-17
- Gerbers regenerated after component renumbering
- README rewritten for v3 features and new designators

Co-Authored-By: Claude Sonnet 4.6 <noreply@anthropic.com>
Parts:
- added D1, D2, D3, D4: GREEN, LED_SMD:LED_0603_1608Metric, symbol Device:LED
- added R1, R2, R3, R4: 330, Resistor_SMD:R_0402_1005Metric, symbol Device:R
- added R10, R11, R12, R13, R14, R15, R16, R17, R18, R19, R20, R5, R6, R7, R8, R9: 10K, Resistor_SMD:R_0402_1005Metric, symbol Device:R
- JP1: value SIZE: open=8MB closed=4MB -> MODEL: open=M5120(9MB) closed=M5126(7MB)
- renumbered C4 to C1, C12 to C10, C9 to C11, C18 to C12, C10 to C13, C17 to C14, C14 to C15, C13 to C17, C15 to C18, C3 to C2, C2 to C3, C1 to C4, C8 to C5, C7 to C6, C6 to C7, C5 to C8, C11 to C9, J2 to J1, J1 to J2, R3 to R21, R2 to R22, R4 to R23, R5 to R24, U2 to U1, U11 to U10, U12 to U11, U3 to U2, U4 to U3, U5 to U4, U6 to U5, U7 to U6, U8 to U7, U9 to U8, U1 to U9
Connections:
- net GND: now also D1.1 (K), D2.1 (K), D3.1 (K), D4.1 (K), R10.2, R11.2, R12.2, R13.2, R14.2, R15.2, R16.2, R17.2, R18.2, R19.2, R20.2, R5.2, R6.2, R7.2, R8.2, R9.2
- net SD0: now also R5.1
- net SD1: now also R6.1
- net SD10: now also R15.1
- net SD11: now also R16.1
- net SD12: now also R17.1
- net SD13: now also R18.1
- net SD14: now also R19.1
- net SD15: now also R20.1
- net SD2: now also R7.1
- net SD3: now also R8.1
- net SD4: now also R9.1
- net SD5: now also R10.1
- net SD6: now also R11.1
- net SD7: now also R12.1
- net SD8: now also R13.1
- net SD9: now also R14.1
- net LED0: now reaches U9.35 (I/O/GCLK3)
- net LED0: now also R1.2
- net LED1: now reaches U9.37 (I/GCLK1)
- net LED1: now also R2.2
- net LED2: now reaches U9.38 (I/OE1/Vpp)
- net LED2: now also R3.2
- net LED3: now reaches U9.39 (I/GCLR)
- net LED3: now also R4.2
- net SIZE8 renamed MODEL
- new net: D2.2 (A), R2.1
- new net: D4.2 (A), R4.1
- new net: D3.2 (A), R3.1
- new net: D1.2 (A), R1.1
- no-connect marks 13 -> 9
Other:
- note added: "DESIGN NOTES — v3.0 MEMORY MAP: 4 banks x 2MB (1Mx16 pairs) fill the expansion window 0x100000–0x8FFFFF = 8MB (9MB system total on M5120). Banks straddle even-MB boundaries because the window starts at 1MB. BANKSEL (CPLD pin 33) = !A20 — selects which 1MB half of each 2MB bank is active; drives A19 (pin 18) on all SRAMs. Chip A0–A18 = Mac A1–A19. WRITE ENABLES — DO NOT MERGE: /WE (pin 28) = low b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"
- note added: "MODEL CONFIG"
- note removed: "DESIGN NOTES — v2.0 MEMORY MAP: 4 banks x 2MB (1Mx16 pairs) fill the expansion window 0x100000–0x8FFFFF = 8MB (9MB system total). Banks straddle even-MB boundaries because the window starts at 1MB. BANKSEL (CPLD pin 33) = !A20 — selects which 1MB half of each 2MB bank is active; drives A19 (pin 18) on all SRAMs. Chip A0–A18 = Mac A1–A19. WRITE ENABLES — DO NOT MERGE: /WE (pin 28) = low byte U2–U5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"
- note removed: "SIZE CONFIG"
- moved on the sheet: C1, C11, C12, C13, C14, C15, C17, C18, C2, C3, C4, C5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

Commit message: Fix CPLD LED pin assignments: move LED1/2/3 from dedicated input pins to valid I/O pins
Pins 37/38/39 on ATF1502ASL TQFP-44 are dedicated input-only pins with no output
driver. Declaring registered outputs (LED1/2/3) there caused the fitter to fail all
PREASSIGN=KEEP passes and fall back to IGNORE, scrambling every pin assignment.

- firmware/PortableRAM8.pld: LED1 pin 37->42, LED2 pin 38->43, LED3 pin 39->44
- PortableRAM-8MB.kicad_sch: reconnected LED1/2/3 nets to pins 42/43/44; X on 37/38/39
- PortableRAM-8MB.kicad_pcb: netlist updated, traces rerouted to pads 42/43/44
- firmware/PortableRAM8.jed/.fit/.svf: recompiled; fitter now succeeds PREASSIGN=KEEP

Co-Authored-By: Claude Sonnet 4.6 <noreply@anthropic.com>
Connections:
- net LED1: now also U9.42 (I/O); no longer U9.37 (I/GCLK1)
- net LED2: now also U9.43 (I/O); no longer U9.38 (I/OE1/Vpp)
- net LED3: now also U9.44 (I/O); no longer U9.39 (I/GCLR)
Changed lines of the file:
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@@
 		)
 	)
-	(text "DESIGN NOTES — v3.0\n\nMEMORY MAP: 4 banks x 2MB (1Mx16 pairs) fill the expansion window\n0x100000–0x8FFFFF = 8MB (9MB system total on M5120). Banks straddle\neven-MB boundaries because the window starts at 1MB.\n\nBANKSEL (CPLD pin 33) = !A20 — selects which 1MB half of each 2MB\nbank is active; drives A19 (pin 18) on all SRAMs.\nChip A0–A18 = Mac A1–A19.\n\nWRITE ENABLES — DO NOT MERGE: /WE (pin 28) = low byte U2–U5,\ngated by /LDS. /WEH (pin 30) = high byte U6–U9, gated by /UDS.\nA common WE corrupts the partner byte on 68000 byte writes.\n\nMODEL JUMPER JP1: OPEN = M5120 non-backlit, all 4 banks active,\n8MB expansion = 9MB total. CLOSED = M5126 backlit, bank 3\n(0x700000–0x8FFFFF) gated off, 6MB expansion = 7MB total.\nAvoids SLOT_CS0 conflict on backlit models above 0x700000.\n\nBANK POPULATION: populate sequentially from bank 0 (U2+U6).\nGhost RAM prevention: R6–R21 (10K pull-downs on data bus, SRAM\nside of 74HC245) ensure empty banks return 0x0000 so Mac boot\nRAM sizing halts cleanly without ghost RAM detection.\n\nSTATUS LEDs (LED0–LED3): CPLD registered outputs (pins 35,37,38,39)\nthat latch ON when Mac boot probe first accesses each bank.\nPower-cycle clears. LED on = bank found and sized at boot.\n330R series resistors (R22–R25).\n\nCS2 (SRAM pin 40): active-high 2nd enable, tied to +5V (unused).\nDTACK: not driven by this card — the Portable's CPU GLU generates it.\nALL-5V DESIGN: no LDO. AS6C8008 are 2.7–5.5V parts."
+	(text "DESIGN NOTES — v3.0\n\nMEMORY MAP: 4 banks x 2MB (1Mx16 pairs) fill the expansion window\n0x100000–0x8FFFFF = 8MB (9MB system total on M5120). Banks straddle\neven-MB boundaries because the window starts at 1MB.\n\nBANKSEL (CPLD pin 33) = !A20 — selects which 1MB half of each 2MB\nbank is active; drives A19 (pin 18) on all SRAMs.\nChip A0–A18 = Mac A1–A19.\n\nWRITE ENABLES — DO NOT MERGE: /WE (pin 28) = low byte U2–U5,\ngated by /LDS. /WEH (pin 30) = high byte U6–U9, gated by /UDS.\nA common WE corrupts the partner byte on 68000 byte writes.\n\nMODEL JUMPER JP1: OPEN = M5120 non-backlit, all 4 banks active,\n8MB expansion = 9MB total. CLOSED = M5126 backlit, bank 3\n(0x700000–0x8FFFFF) gated off, 6MB expansion = 7MB total.\nAvoids SLOT_CS0 conflict on backlit models above 0x700000.\n\nBANK POPULATION: populate sequentially from bank 0 (U2+U6).\nGhost RAM prevention: R6–R21 (10K pull-downs on data bus, SRAM\nside of 74HC245) ensure empty banks return 0x0000 so Mac boot\nRAM sizing halts cleanly without ghost RAM detection.\n\nSTATUS LEDs (LED0–LED3): CPLD registered outputs (pins 35,42,43,44)\nthat latch ON when Mac boot probe first accesses each bank.\nPower-cycle clears. LED on = bank found and sized at boot.\n330R series resistors (R22–R25).\n\nCS2 (SRAM pin 40): active-high 2nd enable, tied to +5V (unused).\nDTACK: not driven by this card — the Portable's CPU GLU generates it.\nALL-5V DESIGN: no LDO. AS6C8008 are 2.7–5.5V parts."
 		(exclude_from_sim no)
 		(at 55 240 0)
@@
 	)
 	(no_connect
-		(at 220.98 69.85)
-	)
-	(no_connect
-		(at 220.98 67.31)
-	)
-	(no_connect
 		(at 215.9 266.7)
 	)
@@
 	)
 	(no_connect
+		(at 220.98 80.01)
+	)
+	(no_connect
 		(at 220.98 74.93)
 	)
 	(no_connect
-		(at 220.98 72.39)
+		(at 220.98 77.47)
 	)
 	(no_connect
@@
 		(at 215.9 261.62)
 	)
+	(no_connect
+		(at 220.98 82.55)
+	)
 	(wire
 		(pts
@@
 		)
 	)
-	(label "LED1"
-		(at 220.98 82.55 0)
-		(effects
-			(font
-				(size 1.27 1.27)
-			)
-			(justify left bottom)
-		)
-	)
 	(label "A16"
 		(at 389.89 104.14 0)
@@
 		)
 	)
+	(label "LED1"
+		(at 220.98 72.39 0)
+		(effects
+			(font
+				(size 1.27 1.27)
+			)
+			(justify left bottom)
+		)
+	)
 	(label "A6"
 		(at 389.89 78.74 0)
@@
 		)
 	)
-	(label "LED3"
-		(at 220.98 77.47 0)
-		(effects
-			(font
-				(size 1.27 1.27)
-			)
-			(justify left bottom)
-		)
-	)
 	(label "SD9"
 		(at 426.72 193.04 0)
@@
 		)
 	)
+	(label "LED3"
+		(at 220.98 67.31 0)
+		(effects
+			(font
+				(size 1.27 1.27)
+			)
+			(justify left bottom)
+		)
+	)
 	(label "A3"
 		(at 389.89 195.58 0)
@@
 		)
 	)
+	(label "LED2"
+		(at 220.98 69.85 0)
+		(effects
+			(font
+				(size 1.27 1.27)
+			)
+			(justify left bottom)
+		)
+	)
 	(label "TDO"
 		(at 226.06 92.71 0)
@@
 		(effects
 			(font
-				(size 1.27 1.27)
-			)
-			(justify left bottom)
-		)
-	)
-	(label "LED2"
-		(at 220.98 80.01 0)
-		(effects
-			(font

Commit message: Add J3 PDS header (1x2, 2.54mm): DTACK→pin 23, EXT_DTACK→pin 31
Schematic: added Conn_01x02 J3 with nets DTACK_OUT/EXT_DTACK_OUT
wired to U9 CPLD pins 23 and 31. Removed no-connect markers from
those pads.

PCB: placed J3 on board edge, routed U9 pad 23→J3 pin 1 (DTACK)
and U9 pad 31→J3 pin 2 (EXT_DTACK). DRC clean: 0 errors,
0 unconnected pads.

User connects J3 pin 1 to PDS B7 (/DTACK) with a removable wire.
No more soldering to CPLD pads.

Co-Authored-By: Claude Sonnet 4.6 <noreply@anthropic.com>
Parts:
- added J3: PDS Header 1x2, Connector_PinHeader_2.54mm:PinHeader_1x02_P2.54mm_Vertical, symbol Connector:Conn_01x02_Pin
Connections:
- net DTACK_OUT: now reaches U9.23 (I/O)
- net DTACK_OUT: now also J3.1 (Pin_1)
- net EXT_DTACK_OUT: now reaches U9.31 (I/O)
- net EXT_DTACK_OUT: now also J3.2 (Pin_2)
- no-connect marks 9 -> 7
Other:
- note added: "DTACK Header for PDS Wire"
Changed lines of the file:
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@@
 		)
 	)
+	(text "DTACK Header for PDS Wire"
+		(exclude_from_sim no)
+		(at 179.07 161.29 0)
+		(effects
+			(font
+				(size 2.54 2.54)
+				(thickness 0.508)
+				(bold yes)
+			)
+			(justify left bottom)
+		)
+	)
 	(text "ERC power anchors — +5V / GND arrive via J1\n(PWR_FLAGs tell ERC these rails are driven)"
 		(exclude_from_sim no)
@@
 	)
 	(no_connect
-		(at 220.98 95.25)
-	)
-	(no_connect
 		(at 220.98 80.01)
 	)
@@
 	)
 	(no_connect
-		(at 220.98 110.49)
-	)
-	(no_connect
 		(at 203.2 261.62)
 	)
@@
 		)
 	)
+	(label "DTACK_OUT"
+		(at 220.98 110.49 0)
+		(effects
+			(font
+				(size 1.27 1.27)
+			)
+			(justify left bottom)
+		)
+	)
 	(label "TCK"
 		(at 92.71 162.56 0)
@@
 		)
 	)
+	(label "EXT_DTACK_OUT"
+		(at 220.98 95.25 0)
+		(effects
+			(font
+				(size 1.27 1.27)
+			)
+			(justify left bottom)
+		)
+	)
 	(label "SLEEP"
 		(at 177.8 87.63 0)
@@
 		)
 	)
+	(label "EXT_DTACK_OUT"
+		(at 208.28 173.99 0)
+		(effects
+			(font
+				(size 1.27 1.27)
+			)
+			(justify left bottom)
+		)
+	)
 	(label "SD14"
 		(at 369.57 205.74 0)
@@
 		)
 	)
+	(label "DTACK_OUT"
+		(at 208.28 171.45 0)
+		(effects
+			(font
+				(size 1.27 1.27)
+			)
+			(justify left bottom)
+		)
+	)
 	(label "D7"
 		(at 222.25 276.86 0)
@@
 					(unit 1)
 				)
+			)
+		)
+	)
+	(symbol
+		(lib_id "Connector:Conn_01x02_Pin")
+		(at 203.2 171.45 0)
+		(unit 1)
+		(exclude_from_sim no)
+		(in_bom yes)
+		(on_board yes)
+		(dnp no)
+		(fields_autoplaced yes)
+		(property "Reference" "J3"
+			(at 203.835 166.37 0)
+			(effects
+				(font
+					(size 1.27 1.27)
+				)
+			)
+		)
+		(property "Value" "PDS Header 1x2"
+			(at 203.835 168.91 0)
+			(effects
+				(font
+					(size 1.27 1.27)
+				)
+			)
+		)
+		(property "Footprint" "Connector_PinHeader_2.54mm:PinHeader_1x02_P2.54mm_Vertical"
+			(at 203.2 171.45 0)
+			(effects
+				(font
+					(size 1.27 1.27)
+				)
+				(hide yes)
+			)
+		)
+		(property "Datasheet" "~"
+			(at 203.2 171.45 0)
+			(effects
+				(font
+					(size 1.27 1.27)
+				)
+				(hide yes)
+			)
+		)
+		(property "Description" "Generic connector, single row, 01x02, script generated"
+			(at 203.2 171.45 0)
+			(effects
+				(font
+					(size 1.27 1.27)
+				)
+				(hide yes)
+			)
+		)
+		(pin "1"
+		)
+		(pin "2"
+		)
+		(instances
+			(project "PortableRAM-8MB"
+				(path "/3f227e15-b881-4174-9819-781940a19688"
+					(reference "J3")
+					(unit 1)
+				)

Commit message: fix: swap J1↔J2 to match v2 convention; add J3 to BOM
v3 had J1=JTAG and J2=RAM connector — reversed from v2.
Correct convention (matching v2): J1=RAM connector (Samtec),
J2=JTAG header, J3=DTACK header.

Updated schematic, PCB, BOM CSV, and README throughout.
Also added missing J3 PDS DTACK header row to BOM CSV.

Co-Authored-By: Claude Sonnet 4.6 <noreply@anthropic.com>
Parts:
- renumbered J2 to J1, J1 to J2
Changed lines of the file:
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@@
 		(dnp no)
 		(fields_autoplaced yes)
-		(property "Reference" "J1"
+		(property "Reference" "J2"
 			(at 98.425 154.94 0)
 			(effects
@@
 			(project "PortableRAM-8MB"
 				(path "/3f227e15-b881-4174-9819-781940a19688"
-					(reference "J1")
+					(reference "J2")
 					(unit 1)
 				)
@@
 		(dnp no)
 		(fields_autoplaced yes)
-		(property "Reference" "J2"
+		(property "Reference" "J1"
 			(at 209.55 222.25 0)
 			(effects
@@
 			(project "PortableRAM-8MB"
 				(path "/3f227e15-b881-4174-9819-781940a19688"
-					(reference "J2")
+					(reference "J1")
 					(unit 1)
 				)
